File: kl10/kl10.sch (KiCad schematic (older format))
At the start: 5 parts, among them U1 MC10164

Commit message: checkpoint
Parts:
- added e28, e62, e68: MC10110, symbol MC10110
- added e39, e51: MC10141, symbol MC10141
- added e40, e41, e46, e47, e54: MC10164, symbol MC10164
- gave numbers to parts that had none: 1
- renumbered U1 to e53
Connections:
- net labels added: [n/18+1,ctl.arl.sel.1.h,ctl.arr.sel.1.h], [n/18+1,ctl.arl.sel.2.h,ctl.arr.sel.2.h], [n/18+1,ctl.arl.sel.4.h,cram.arm.sel.4.a.h], [n/30+1,ad.[n+6].h,adx.00.h], [n/6+1,ctl.ar.00-08.load.l,ctl.ar.00-08.load.l,ctl.ar.09-17.load.l,ctl.arr.load.b.l,ctl.arr.load.b.l,ctl.arr.load.b.l], [n/6+1,ctl.ar.00-08.load.l,ctl.ar.09-17.load.l,ctl.ar.09-17.load.l,ctl.arr.load.a.l,ctl.arr.load.a.l,ctl.arr.load.a.l], [n/6+1,ctl.ar.00-11.clr.h,ctl.ar.00-11.clr.h,ctl.ar.12-17.clr.h,ctl.arr.clr.h,ctl.arr.clr.h,ctl.arr.clr.h], [n/b+1],ad.ex.-01.h,ad.05.h,ad.11.h,ad.17.h,ad.23.h,ad.23.h], ad.[n+2].h, ad.[n+3].h, ad.[n+4].h, ad.[n+5].h, adx.[n+1].h, adx.[n+2].h, adx.[n+3].h, adx.[n+5].h, ar.[n+0].a.h, ar.[n+0].b.h, ar.[n+0].c.h, ar.[n+0].d.h, ar.[n+0].h, ar.[n+1].a.h, ar.[n+1].b.h, ar.[n+1].c.h, ar.[n+1].h, ar.[n+2].a.h, ar.[n+2].b.h, ar.[n+2].c.h, ar.[n+2].h, ar.[n+3].a.h, ar.[n+3].b.h, ar.[n+3].c.h, ar.[n+3].h, ar.[n+4].a.h, ar.[n+4].b.h, ar.[n+4].c.h, ar.[n+4].h, ar.[n+5].a.h, ar.[n+5].b.h, ar.[n+5].c.h, ar.[n+5].h, arm.[n+0].h, arm.[n+1].h, arm.[n+2].h, arm.[n+3].h, arm.[n+4].h, arm.[n+5].h, armm.[n+1].h, armm.[n+2].h, armm.[n+3].h, armm.[n+4].h, armm.[n+5].h, cache.data.[n+1].b.h, cache.data.[n+2].b.h, cache.data.[n+3].b.h, cache.data.[n+4].b.h, cache.data.[n+5].b.h, dp04.clk.b.h, dp04.clk.f.h, ebus.d[n+1].e.h, ebus.d[n+2].e.h, ebus.d[n+3].e.h, ebus.d[n+4].e.h, ebus.d[n+5].e.h, sh.[n+1].h, sh.[n+2].h, sh.[n+3].h, sh.[n+4].h, sh.[n+5].h
- wire segments 19 -> 144
- no-connect marks 0 -> 26
Other:
- moved on the sheet: e52A, e52B, e52C, e52D, e53

Commit message: checkpoint
Parts:
- added e? (x6): MC10164, symbol MC10164
- added e? (x4): MC10101, symbol MC10101
- added e? (x2): MC10141, symbol MC10141
- added e? (x6): MC10110, symbol MC10110
Connections:
- wire segments 144 -> 288
- no-connect marks 26 -> 52

Commit message: checkpoint
Parts:
- removed e28, e62, e68, e? (x6): MC10110, symbol MC10110
- removed e39, e51, e? (x2): MC10141, symbol MC10141
- removed e40, e41, e46, e47, e53, e54, e? (x6): MC10164, symbol MC10164
- removed e52, e? (x4): MC10101, symbol MC10101
Connections:
- no-connect marks 52 -> 8
