File: kl10/dpa.sch (KiCad schematic (older format))
At the start: 8 parts

Commit message: checkpoint
Parts:
- removed e39, e51: MC10141, symbol MC10141
- removed e40, e41, e46, e47, e53, e54: MC10164, symbol MC10164
Connections:
- net labels removed: ad, ad.0, ad.1, ad.2, ad.3, ad.4, ad.5, adx.0, adx.1, adx.2, adx.3, adx.4, adx.5, ar, ar-0-2-sel, ar-3-5-sel, ar.0, ar.1, ar.2, ar.3, ar.4, ar.5, arm-en, arm-sel-1, arm-sel-2, arm-sel-4, arm.0, arm.0-x7, arm.1, arm.1-x7, arm.2, arm.3, arm.4, arm.4-x5, arm.5, arm.5-x5, armm, armm.0, armm.1, armm.2, armm.3, armm.4, armm.5, cache-data, cache-data.0, cache-data.1, cache-data.2, cache-data.3, cache-data.4, cache-data.5, dp04-clk, ebus-d, ebus-d.0, ebus-d.1, ebus-d.2, ebus-d.3, ebus-d.4, ebus-d.5, sh, sh.0, sh.1, sh.2, sh.3, sh.4, sh.5
- wire segments 133 -> 0
- no-connect marks 12 -> 0

Commit message: DPA seems to be "done-ish"
Changed lines of the file:
@@
 F1 "dpa01.sch" 60
 F2 "dp04-clk" I L 2050 2650 60
-F3 "ar" O R 3200 2650 60
-F4 "armm" I L 2050 4500 60
-F5 "ad" I L 2050 4400 60
-F6 "cache-data" I L 2050 4100 60
-F7 "ebus-d" I L 2050 4200 60
-F8 "sh" I L 2050 4600 60
-F9 "[n/6+1,ctl-ar-00-08-load l,ctl-ar-00-08-load-l,ctl-ar-09-17-load-l,ctl-arr-load-l,ctl-arr-load-l,ctl-arr-load-l]" I L 2050 4700 60
-F10 "[n/6+1,ctl-ar-00-08-load-l,ctl-ar-09-17-load-l,ctl-ar-09-17-load-l,ctl-arr-load-l,ctl-arr-load-l,ctl-arr-load-l]" I L 2050 4800 60
-F11 "[n/18+1,ctl-arl-sel-4,cram-arm-sel-4]" I L 2050 4900 60
-F12 "[n/18+1,ctl-arl-sel-2,ctl-arr-sel-2]" I L 2050 5000 60
+F3 "[n/6+1,ctl-ar-00-08-load l,ctl-ar-00-08-load-l,ctl-ar-09-17-load-l,ctl-arr-load-l,ctl-arr-load-l,ctl-arr-load-l]" I L 2050 4700 60
+F4 "[n/6+1,ctl-ar-00-08-load-l,ctl-ar-09-17-load-l,ctl-ar-09-17-load-l,ctl-arr-load-l,ctl-arr-load-l,ctl-arr-load-l]" I L 2050 4800 60
+F5 "[n/18+1,ctl-arl-sel-4,cram-arm-sel-4]" I L 2050 4900 60
+F6 "[n/18+1,ctl-arl-sel-2,ctl-arr-sel-2]" I L 2050 5000 60
 $EndSheet
 $Sheet

Commit message: Update to kicad 5.1.2
Changed lines of the file:
@@
-EESchema Schematic File Version 2
-LIBS:o_ecl
-LIBS:ecl
-LIBS:power
-LIBS:device
-LIBS:transistors
-LIBS:conn
-LIBS:linear
-LIBS:regul
-LIBS:74xx
-LIBS:cmos4000
-LIBS:adc-dac
-LIBS:memory
-LIBS:xilinx
-LIBS:microcontrollers
-LIBS:dsp
-LIBS:microchip
-LIBS:analog_switches
-LIBS:motorola
-LIBS:texas
-LIBS:intel
-LIBS:audio
-LIBS:interface
-LIBS:digital-audio
-LIBS:philips
-LIBS:display
-LIBS:cypress
-LIBS:siliconi
-LIBS:opto
-LIBS:atmel
-LIBS:contrib
-LIBS:valves
+EESchema Schematic File Version 4
 LIBS:kl10-cache
-EELAYER 25 0
+EELAYER 30 0
 EELAYER END
 $Descr B 17000 11000
@@
 	1900 2650 2050 2650
 Wire Wire Line
-	1700 2250 13500 2250
+	1700 2250 1900 2250
 Wire Wire Line
 	5250 2250 5250 2650
@@
 Text HLabel 13200 3200 0    60   Input ~ 0
 adx
+Wire Wire Line
+	1900 2250 5250 2250
+Wire Wire Line
+	5250 2250 13500 2250
 $EndSCHEMATC
