File: kl10/dpa01.sch (KiCad schematic (older format))
At the start: 8 parts

Commit message: checkpoint
Connections:
- net labels added: [n/18+1,ctl-arl-sel-1,ctl-arr-sel-1], [n/18+1,ctl-arl-sel-2,ctl-arr-sel-2], [n/18+1,ctl-arl-sel-4,cram-arm-sel-4], [n/30+1,ad.[n+6],adx.0], [n/6+1,ad-ex.1,ad.5,ad.11,ad.17,ad.23,ad.29], [n/6+1,ad-ex.2,ad.4,ad.10,ad.16,ad.22,ad.28], [n/6+1,ctl-ar-00-08-load l,ctl-ar-00-08-load-l,ctl-ar-09-17-load-l,ctl-arr-load-l,ctl-arr-load-l,ctl-arr-load-l], [n/6+1,ctl-ar-00-08-load-l,ctl-ar-09-17-load-l,ctl-ar-09-17-load-l,ctl-arr-load-l,ctl-arr-load-l,ctl-arr-load-l], [n/6+1,ctl-ar-00-11-clr,ctl-ar-00-11-clr,ctl-ar-12-17-clr,ctl-arr-clr,ctl-arr-clr,ctl-arr-clr]
- net labels removed: ar-0-2-sel, ar-3-5-sel, arm-en, arm-sel-1, arm-sel-2, arm-sel-4, arm.0-x7, arm.1-x7, arm.4-x5, arm.5-x5
Changed lines of the file:
@@
 U 1 1 57A676FA
 P 3900 3600
+AR Path="/57B68864/57B6B963/57A676FA" Ref="e53"  Part="1"
+AR Path="/57B6D511/57B6B963/57A676FA" Ref="e53"  Part="1"
 F 0 "e53" H 3920 4350 60  0000 C CNN
 F 1 "MC10164" H 3940 2850 60  0000 C CNN
@@
 U 1 1 57A7828A
 P 7050 3600
+AR Path="/57B68864/57B6B963/57A7828A" Ref="e46"  Part="1"
+AR Path="/57B6D511/57B6B963/57A7828A" Ref="e46"  Part="1"
 F 0 "e46" H 7070 4350 60  0000 C CNN
 F 1 "MC10164" H 7090 2850 60  0000 C CNN
@@
 U 1 1 57A791AF
 P 10150 3600
+AR Path="/57B68864/57B6B963/57A791AF" Ref="e47"  Part="1"
+AR Path="/57B6D511/57B6B963/57A791AF" Ref="e47"  Part="1"
 F 0 "e47" H 10170 4350 60  0000 C CNN
 F 1 "MC10164" H 10190 2850 60  0000 C CNN
@@
 U 1 1 57A7ADE0
 P 12050 1900
+AR Path="/57B68864/57B6B963/57A7ADE0" Ref="e39"  Part="1"
+AR Path="/57B6D511/57B6B963/57A7ADE0" Ref="e39"  Part="1"
 F 0 "e39" H 12070 2500 60  0000 C CNN
 F 1 "MC10141" H 12090 1300 60  0000 C CNN
@@
 U 1 1 57A7DDB6
 P 4150 8950
+AR Path="/57B68864/57B6B963/57A7DDB6" Ref="e41"  Part="1"
+AR Path="/57B6D511/57B6B963/57A7DDB6" Ref="e41"  Part="1"
 F 0 "e41" H 4170 9700 60  0000 C CNN
 F 1 "MC10164" H 4190 8200 60  0000 C CNN
@@
 U 1 1 57A7DDD2
 P 7300 8950
+AR Path="/57B68864/57B6B963/57A7DDD2" Ref="e40"  Part="1"
+AR Path="/57B6D511/57B6B963/57A7DDD2" Ref="e40"  Part="1"
 F 0 "e40" H 7320 9700 60  0000 C CNN
 F 1 "MC10164" H 7340 8200 60  0000 C CNN
@@
 U 1 1 57A7DDF0
 P 10400 8950
+AR Path="/57B68864/57B6B963/57A7DDF0" Ref="e54"  Part="1"
+AR Path="/57B6D511/57B6B963/57A7DDF0" Ref="e54"  Part="1"
 F 0 "e54" H 10420 9700 60  0000 C CNN
 F 1 "MC10164" H 10440 8200 60  0000 C CNN
@@
 U 1 1 57A7DE0C
 P 12300 7250
+AR Path="/57B68864/57B6B963/57A7DE0C" Ref="e51"  Part="1"
+AR Path="/57B6D511/57B6B963/57A7DE0C" Ref="e51"  Part="1"
 F 0 "e51" H 12320 7850 60  0000 C CNN
 F 1 "MC10141" H 12340 6650 60  0000 C CNN
@@
 NoConn ~ 16700 3000
 Text HLabel 10250 2450 0    60   Input ~ 0
-ar-0-2-sel
+[n/6+1,ctl-ar-00-08-load l,ctl-ar-00-08-load-l,ctl-ar-09-17-load-l,ctl-arr-load-l,ctl-arr-load-l,ctl-arr-load-l]
 Text HLabel 10200 2150 0    60   Input ~ 0
 dp04-clk
 Text HLabel 10450 7850 0    60   Input ~ 0
-ar-3-5-sel
+[n/6+1,ctl-ar-00-08-load-l,ctl-ar-09-17-load-l,ctl-ar-09-17-load-l,ctl-arr-load-l,ctl-arr-load-l,ctl-arr-load-l]
 Text HLabel 10450 7500 0    60   Input ~ 0
 dp04-clk
 Text HLabel 2700 4800 0    60   Input ~ 0
-arm-sel-4
+[n/18+1,ctl-arl-sel-4,cram-arm-sel-4]
 Text HLabel 2700 5550 0    60   Input ~ 0
-arm-sel-2
+[n/18+1,ctl-arl-sel-2,ctl-arr-sel-2]
 Text HLabel 2650 6200 0    60   Input ~ 0
-arm-sel-1
+[n/18+1,ctl-arl-sel-1,ctl-arr-sel-1]
 Text HLabel 2650 6850 0    60   Input ~ 0
-arm-en
+[n/6+1,ctl-ar-00-11-clr,ctl-ar-00-11-clr,ctl-ar-12-17-clr,ctl-arr-clr,ctl-arr-clr,ctl-arr-clr]
 Wire Wire Line
 	4500 3000 4500 1650
@@
 ad.3
 Text HLabel 9700 8850 0    60   Input ~ 0
-arm.5-x5
+[n/30+1,ad.[n+6],adx.0]
 Text HLabel 6350 3700 0    60   Input ~ 0
-arm.1-x7
+[n/6+1,ad-ex.1,ad.5,ad.11,ad.17,ad.23,ad.29]
 Text HLabel 3250 3700 0    60   Input ~ 0
-arm.0-x7
+[n/6+1,ad-ex.2,ad.4,ad.10,ad.16,ad.22,ad.28]
 Text Label 6600 8350 2    60   ~ 0
 armm.4
@@
 Text Label 6600 9050 2    60   ~ 0
 ad.2
-Text HLabel 6600 8850 0    60   Input ~ 0
-arm.4-x5
 Text Label 2600 8350 2    60   ~ 0
 armm.4
@@
 Text HLabel 1800 2900 0    60   Input ~ 0
 sh
+Text Label 6600 8850 2    60   ~ 0
+ad.5
 $EndSCHEMATC

Commit message: DPA seems to be "done-ish"
Connections:
- net labels added: ad.[n+0], ad.[n+1], ad.[n+2], ad.[n+3], ad.[n+4], ad.[n+5], adx.[n+0], adx.[n+1], adx.[n+2], adx.[n+3], adx.[n+4], adx.[n+5], ar.[n+0], ar.[n+1], ar.[n+2], ar.[n+3], ar.[n+4], ar.[n+5], arm.[n+0], arm.[n+1], arm.[n+2], arm.[n+3], arm.[n+4], arm.[n+5], armm.[n+0], armm.[n+1], armm.[n+4], armm.[n+5], armm.[n+[n]+2], cache-data.[n+0], cache-data.[n+1], cache-data.[n+2], cache-data.[n+3], cache-data.[n+4], cache-data.[n+5], ebus-d.[n+0], ebus-d.[n+1], ebus-d.[n+2], ebus-d.[n+3], ebus-d.[n+4], ebus-d.[n+5], sh.[n+0], sh.[n+1], sh.[n+2], sh.[n+3], sh.[n+4], sh.[n+5]
- net labels removed: ad, ad.0, ad.1, ad.2, ad.3, ad.4, ad.5, adx.0, adx.1, adx.2, adx.3, adx.4, adx.5, ar, ar.0, ar.1, ar.2, ar.3, ar.4, ar.5, arm.0, arm.1, arm.2, arm.3, arm.4, arm.5, armm, armm.0, armm.1, armm.2, armm.3, armm.4, armm.5, cache-data, cache-data.0, cache-data.1, cache-data.2, cache-data.3, cache-data.4, cache-data.5, ebus-d, ebus-d.0, ebus-d.1, ebus-d.2, ebus-d.3, ebus-d.4, ebus-d.5, sh, sh.0, sh.1, sh.2, sh.3, sh.4, sh.5
- wire segments 133 -> 96

Commit message: Update to kicad 5.1.2
Parts:
- e39, e51: symbol MC10141 -> o_ecl:MC10141
- e40, e41, e46, e47, e53, e54: symbol MC10164 -> o_ecl:MC10164
Changed lines of the file:
@@
-EESchema Schematic File Version 2
-LIBS:o_ecl
-LIBS:ecl
-LIBS:power
-LIBS:device
-LIBS:transistors
-LIBS:conn
-LIBS:linear
-LIBS:regul
-LIBS:74xx
-LIBS:cmos4000
-LIBS:adc-dac
-LIBS:memory
-LIBS:xilinx
-LIBS:microcontrollers
-LIBS:dsp
-LIBS:microchip
-LIBS:analog_switches
-LIBS:motorola
-LIBS:texas
-LIBS:intel
-LIBS:audio
-LIBS:interface
-LIBS:digital-audio
-LIBS:philips
-LIBS:display
-LIBS:cypress
-LIBS:siliconi
-LIBS:opto
-LIBS:atmel
-LIBS:contrib
-LIBS:valves
+EESchema Schematic File Version 4
 LIBS:kl10-cache
-EELAYER 25 0
+EELAYER 30 0
 EELAYER END
 $Descr B 17000 11000
@@
 $EndDescr
 $Comp
-L MC10164 e53
+L o_ecl:MC10164 e53
 U 1 1 57A676FA
 P 3900 3600
@@
 	2850 4100 3300 4100
 $Comp
-L MC10164 e46
+L o_ecl:MC10164 e46
 U 1 1 57A7828A
 P 7050 3600
@@
 	7650 3000 7800 3000
 $Comp
-L MC10164 e47
+L o_ecl:MC10164 e47
 U 1 1 57A791AF
 P 10150 3600
@@
 Connection ~ 6450 4200
 $Comp
-L MC10141 e39
+L o_ecl:MC10141 e39
 U 1 1 57A7ADE0
 P 12050 1900
@@
 	10200 2150 11450 2150
 $Comp
-L MC10164 e41
+L o_ecl:MC10164 e41
 U 1 1 57A7DDB6
 P 4150 8950
@@
 	2600 8950 3550 8950
 $Comp
-L MC10164 e40
+L o_ecl:MC10164 e40
 U 1 1 57A7DDD2
 P 7300 8950
@@
 	7900 8350 8050 8350
 $Comp
-L MC10164 e54
+L o_ecl:MC10164 e54
 U 1 1 57A7DDF0
 P 10400 8950
@@
 Connection ~ 6700 9550
 $Comp
-L MC10141 e51
+L o_ecl:MC10141 e51
 U 1 1 57A7DE0C
 P 12300 7250
