File: kl10/dpa03.sch (KiCad schematic (older format))
At the start: 1 part

Commit message: checkpoint
Parts:
- added e12, e14, e16, e18, e19, e23, e26, e6, e9: MC10174, symbol MC10174
- added e17, e5: MC10158, symbol MC10158
- added e2, e3, e4: MC10181, symbol MC10181
- added e21, e22: MC10164, symbol MC10164
- added e29: MC10105, symbol MC10105
- added e33: MC10107, symbol MC10107
- added e7: MC10109, symbol MC10109
- gave numbers to parts that had none: 1
Connections:
- net labels added: #.0, #.1, #.2, #.3, #.4, #.5, ad-2-5-cin, ad-cg.2, ad-cg.3, ad-cp.2, ad-cp.3, ad-cry.1, ad-cry.1-l, ad-ex.-1, ad-overflow.0-l, ad.0-5=0, ada.2, ada.3, ada.4, ada.5, adb.-2-sel4, adb.2, adb.3, adb.4, adb.4-d03, adb.5, adb.5-d11, adb.5-d13, adx-3-5-cin, adx-cry.3, adx.0, adx.1, adx.2, adx.3, adx.4, adx.5, adxa.0, adxa.1, adxa.2, adxa.3, adxa.4, adxa.5, adxb.0, adxb.1, adxb.2, adxb.3, adxb.4, adxb.5, arx.6, brx.6, brx.7, cram-ada-dis.0, cram-ada-sel1, cram-ada-sel2, cram-adb-sel1, cram-adb-sel2
- net labels removed: ad-ex.1, ad-ex.2
- wire segments 17 -> 108
- no-connect marks 0 -> 30
Other:
- moved on the sheet: e1

Commit message: DPA seems to be "done-ish"
Connections:
- net #.0 renamed #.[n+0]
- net #.1 renamed #.[n+1]
- net #.2 renamed #.[n+2]
- net #.3 renamed #.[n+3]
- net #.4 renamed #.[n+4]
- net #.5 renamed #.[n+5]
- net ad-cg.0 renamed ad-cg.[n+0]
- net ad-cg.2 renamed ad-cg.[n+2]
- net ad-cg.3 renamed ad-cg.[n+3]
- net ad-cp.0 renamed ad-cp.[n+0]
- net ad-cp.2 renamed ad-cp.[n+2]
- net ad-cp.3 renamed ad-cp.[n+3]
- net ad-cry.-2 renamed ad-cry.[n+-2]
- net ad-cry.1 renamed ad-cry.[n+1]
- net ad-cry.1-l renamed ad-cry.[n+1]-l
- net ad-cry.2 renamed ad-cry.[n+2]
- net ad-ex.-1 renamed ad-ex.[n+-1]
- net ad-ex.-2 renamed ad-ex.[n+-2]
- net ad-overflow.0-l renamed ad-overflow.[n+0]-l
- net ad.0 renamed ad.[n+0]
- net ad.0-5=0 renamed ad.[n+0]-[n+5]=0
- net ad.1 renamed ad.[n+1]
- net ad.2 renamed ad.[n+2]
- net ad.3 renamed ad.[n+3]
- net ad.4 renamed ad.[n+4]
- net ad.5 renamed ad.[n+5]
- net ada.0 renamed ada.[n+0]
- net ada.1 renamed ada.[n+1]
- net ada.2 renamed ada.[n+2]
- net ada.3 renamed ada.[n+3]
- net ada.4 renamed ada.[n+4]
- net ada.5 renamed ada.[n+5]
- net adb.-1 renamed adb.[n+-1]
- net adb.-2 renamed adb.[n+-2]
- net adb.-2-sel4 renamed adb.[n+-2]-sel4
- net adb.0 renamed adb.[n+0]
- net adb.1 renamed adb.[n+1]
- net adb.2 renamed adb.[n+2]
- net adb.3 renamed adb.[n+3]
- net adb.4 renamed adb.[n+4]
- net adb.4-d03 renamed adb.[n+4]-d03
- net adb.5 renamed adb.[n+5]
- net adb.5-d11 renamed adb.[n+5]-d11
- net adb.5-d13 renamed adb.[n+5]-d13
- net adx-cry.3 renamed adx-cry.[n+3]
- net adx.0 renamed adx.[n+0]
- net adx.1 renamed adx.[n+1]
- net adx.2 renamed adx.[n+2]
- net adx.3 renamed adx.[n+3]
- net adx.4 renamed adx.[n+4]
- net adx.5 renamed adx.[n+5]
- net adxa.0 renamed adxa.[n+0]
- net adxa.1 renamed adxa.[n+1]
- net adxa.2 renamed adxa.[n+2]
- net adxa.3 renamed adxa.[n+3]
- net adxa.4 renamed adxa.[n+4]
- net adxa.5 renamed adxa.[n+5]
- net adxb.0 renamed adxb.[n+0]
- net adxb.1 renamed adxb.[n+1]
- net adxb.2 renamed adxb.[n+2]
- net adxb.3 renamed adxb.[n+3]
- net adxb.4 renamed adxb.[n+4]
- net adxb.5 renamed adxb.[n+5]
- net ar.0 renamed ar.[n+0]
- net ar.1 renamed ar.[n+1]
- net ar.2 renamed ar.[n+2]
- net ar.3 renamed ar.[n+3]
- net ar.4 renamed ar.[n+4]
- net ar.5 renamed ar.[n+5]
- net arx.0 renamed arx.[n+0]
- net arx.1 renamed arx.[n+1]
- net arx.2 renamed arx.[n+2]
- net arx.3 renamed arx.[n+3]
- net arx.4 renamed arx.[n+4]
- net arx.5 renamed arx.[n+5]
- net arx.6 renamed arx.[n+6]
- net br.0 renamed br.[n+0]
- net br.1 renamed br.[n+1]
- net br.2 renamed br.[n+2]
- net br.3 renamed br.[n+3]
- net br.4 renamed br.[n+4]
- net br.5 renamed br.[n+5]
- net brx.0 renamed brx.[n+0]
- net brx.1 renamed brx.[n+1]
- net brx.2 renamed brx.[n+2]
- net brx.3 renamed brx.[n+3]
- net brx.4 renamed brx.[n+4]
- net brx.5 renamed brx.[n+5]
- net brx.6 renamed brx.[n+6]
- net brx.7 renamed brx.[n+7]
- net cram-ada-dis.0 renamed cram-ada-dis.[n+0]
- net fm.0 renamed fm.[n+0]
- net fm.1 renamed fm.[n+1]
- net fm.2 renamed fm.[n+2]
- net fm.3 renamed fm.[n+3]
- net fm.4 renamed fm.[n+4]
- net fm.5 renamed fm.[n+5]
- net mq.0 renamed mq.[n+0]
- net mq.1 renamed mq.[n+1]
- net mq.2 renamed mq.[n+2]
- net mq.3 renamed mq.[n+3]
- net mq.4 renamed mq.[n+4]
- net mq.5 renamed mq.[n+5]
- net vma-held-or-pc.0 renamed vma-held-or-pc.[n+0]
- net vma-held-or-pc.1 renamed vma-held-or-pc.[n+1]
- net vma-held-or-pc.2 renamed vma-held-or-pc.[n+2]
- net vma-held-or-pc.3 renamed vma-held-or-pc.[n+3]
- net vma-held-or-pc.4 renamed vma-held-or-pc.[n+4]
- net vma-held-or-pc.5 renamed vma-held-or-pc.[n+5]

Commit message: Put back [n...] exprs
Connections:
- net adb.[n+-2]-sel4: no longer e21.10 (C)
- net ad-2-5-cin renamed [n/30+1,ad-cry.[n+6],ad-cry-36]
- net adb.[n+4]-d03 renamed [n/30+1,AR.[n+6],arx.0]
- net adb.[n+5]-d11 renamed [n/30+1,br.[n+6],brx.0]
- net adb.[n+5]-d13 renamed [n/30+1,ar.[n+7],arx.1]
- net adx-3-5-cin renamed [n/30+1,adx-cry.[n+6],ctl-adx-cry-36]
- new net [(n+199)/100,HI,NC]: e21.10 (C)
Changed lines of the file:
@@
 ada.[n+2]
 Text HLabel 6100 3600 0    60   Input ~ 0
-ad-2-5-cin
+[n/30+1,ad-cry.[n+6],ad-cry-36]
 $Comp
 L MC10181 e3
@@
 NoConn ~ 12950 2900
 Text HLabel 11500 3600 0    60   Input ~ 0
-adx-3-5-cin
+[n/30+1,adx-cry.[n+6],ctl-adx-cry-36]
 Text HLabel 13050 3500 2    60   Input ~ 0
 adx-cry.[n+3]
@@
 cram-adb-sel2
 Text HLabel 4600 6150 0    60   Input ~ 0
-adb.[n+-2]-sel4
+[(n+199)/100,HI,NC]
 Text HLabel 4600 5950 0    60   Input ~ 0
 cram-adb-sel1
@@
 adb.[n+5]
 Text HLabel 6700 7350 0    60   Input ~ 0
-adb.[n+4]-d03
+[n/30+1,AR.[n+6],arx.0]
 Text HLabel 6700 7550 0    60   Input ~ 0
-adb.[n+5]-d11
+[n/30+1,br.[n+6],brx.0]
 Text HLabel 6700 7750 0    60   Input ~ 0
-adb.[n+5]-d13
+[n/30+1,ar.[n+7],arx.1]
 $Comp
 L MC10174 e9

Commit message: Update to kicad 5.1.2
Parts:
- e1, e2, e3, e4: symbol MC10181 -> o_ecl:MC10181
- e12, e14, e16, e18, e19, e23, e26, e6, e9: symbol MC10174 -> o_ecl:MC10174
- e17, e5: symbol MC10158 -> o_ecl:MC10158
- e21, e22: symbol MC10164 -> o_ecl:MC10164
- e29: symbol MC10105 -> o_ecl:MC10105
- e33: symbol MC10107 -> o_ecl:MC10107
- e7: symbol MC10109 -> o_ecl:MC10109
Changed lines of the file:
@@
-EESchema Schematic File Version 2
-LIBS:o_ecl
-LIBS:ecl
-LIBS:power
-LIBS:device
-LIBS:transistors
-LIBS:conn
-LIBS:linear
-LIBS:regul
-LIBS:74xx
-LIBS:cmos4000
-LIBS:adc-dac
-LIBS:memory
-LIBS:xilinx
-LIBS:microcontrollers
-LIBS:dsp
-LIBS:microchip
-LIBS:analog_switches
-LIBS:motorola
-LIBS:texas
-LIBS:intel
-LIBS:audio
-LIBS:interface
-LIBS:digital-audio
-LIBS:philips
-LIBS:display
-LIBS:cypress
-LIBS:siliconi
-LIBS:opto
-LIBS:atmel
-LIBS:contrib
-LIBS:valves
+EESchema Schematic File Version 4
 LIBS:kl10-cache
-EELAYER 25 0
+EELAYER 30 0
 EELAYER END
 $Descr B 17000 11000
@@
 $EndDescr
 $Comp
-L MC10181 e1
+L o_ecl:MC10181 e1
 U 1 1 57ACC3A9
 P 4200 3400
@@
 ad.[n+1]
 $Comp
-L MC10181 e2
+L o_ecl:MC10181 e2
 U 1 1 57B4AC90
 P 6850 3400
@@
 [n/30+1,ad-cry.[n+6],ad-cry-36]
 $Comp
-L MC10181 e3
+L o_ecl:MC10181 e3
 U 1 1 57B4BAC9
 P 9550 3400
@@
 NoConn ~ 10250 2900
 $Comp
-L MC10181 e4
+L o_ecl:MC10181 e4
 U 1 1 57B4C236
 P 12250 3400
@@
 adx-cry.[n+3]
 $Comp
-L MC10107 e33
+L o_ecl:MC10107 e33
 U 1 1 57B4D96A
 P 3450 800
@@
 $EndComp
 $Comp
-L MC10105 e29
+L o_ecl:MC10105 e29
 U 3 1 57B4D989
 P 4800 1000
@@
 $EndComp
 $Comp
-L MC10107 e33
+L o_ecl:MC10107 e33
 U 2 1 57B4D9BA
 P 3450 1500
@@
 $EndComp
 $Comp
-L MC10107 e33
+L o_ecl:MC10107 e33
 U 3 1 57B4DC20
 P 4800 1700
@@
 ad-cry.[n+-2]
 $Comp
-L MC10109 e7
+L o_ecl:MC10109 e7
 U 2 1 57B515E0
 P 8850 900
@@
 $EndComp
 $Comp
-L MC10109 e7
+L o_ecl:MC10109 e7
 U 1 1 57B51998
 P 7550 1600
@@
 ad.[n+0]-[n+5]=0
 $Comp
-L MC10164 e22
+L o_ecl:MC10164 e22
 U 1 1 57B53A7D
 P 3250 5650
@@
 adb.[n+-2]
 $Comp
-L MC10164 e21
+L o_ecl:MC10164 e21
 U 1 1 57B54C8B
 P 5200 5650
@@
 adb.[n+-1]
 $Comp
-L MC10174 e14
+L o_ecl:MC10174 e14
 U 1 1 57B565E8
 P 7800 5500
@@
 ada.[n+1]
 $Comp
-L MC10174 e16
+L o_ecl:MC10174 e16
 U 1 1 57B574E0
 P 10400 5500
@@
 ada.[n+3]
 $Comp
-L MC10174 e18
+L o_ecl:MC10174 e18
 U 1 1 57B57BA7
 P 13050 5500
@@
 cram-ad-boole
 $Comp
-L MC10158 e17
+L o_ecl:MC10158 e17
 U 1 1 57B58502
 P 15050 3100
@@
 adxa.[n+2]
 $Comp
-L MC10158 e5
+L o_ecl:MC10158 e5
 U 1 1 57B590AD
 P 15050 1500
@@
 adxa.[n+5]
 $Comp
-L MC10174 e23
+L o_ecl:MC10174 e23
 U 1 1 57B59E83
 P 2400 7550
@@
 adb.[n+1]
 $Comp
-L MC10174 e26
+L o_ecl:MC10174 e26
 U 1 1 57B5AE9B
 P 4800 7550
@@
 adb.[n+3]
 $Comp
-L MC10174 e19
+L o_ecl:MC10174 e19
 U 1 1 57B5B5EA
 P 7300 7550
@@
 [n/30+1,ar.[n+7],arx.1]
 $Comp
-L MC10174 e9
+L o_ecl:MC10174 e9
 U 1 1 57B5C580
 P 9650 7550
@@
 brx.[n+3]
 $Comp
-L MC10174 e12
+L o_ecl:MC10174 e12
 U 1 1 57B5CF64
 P 12050 7550
@@
 brx.[n+5]
 $Comp
-L MC10174 e6
+L o_ecl:MC10174 e6
 U 1 1 57B5D8E4
 P 14500 7550
