File: kl10/dpa04.sch (KiCad schematic (older format))
At the start: 22 parts

Commit message: checkpoint
Changed lines of the file:
@@
 $Descr B 17000 11000
 encoding utf-8
-Sheet 5 6
+Sheet 6 6
 Title "DATA PATH EBUS, FM, BR, BRX"
 Date "10/21/1976"
@@
 U 1 1 57B64287
 P 2750 3650
+AR Path="/57B68864/57B6BA75/57B64287" Ref="e59"  Part="1"
+AR Path="/57B6D511/57B6BA75/57B64287" Ref="e59"  Part="1"
 F 0 "e59" H 2770 3900 60  0000 C CNN
 F 1 "MC10101" H 2790 3400 60  0000 C CNN
@@
 U 2 1 57B6430A
 P 2750 4350
+AR Path="/57B68864/57B6BA75/57B6430A" Ref="e59"  Part="2"
+AR Path="/57B6D511/57B6BA75/57B6430A" Ref="e59"  Part="2"
 F 0 "e59" H 2770 4600 60  0000 C CNN
 F 1 "MC10101" H 2790 4100 60  0000 C CNN
@@
 U 3 1 57B64349
 P 2750 5050
+AR Path="/57B68864/57B6BA75/57B64349" Ref="e59"  Part="3"
+AR Path="/57B6D511/57B6BA75/57B64349" Ref="e59"  Part="3"
 F 0 "e59" H 2770 5300 60  0000 C CNN
 F 1 "MC10101" H 2790 4800 60  0000 C CNN
@@
 U 4 1 57B6437D
 P 2750 5750
+AR Path="/57B68864/57B6BA75/57B6437D" Ref="e59"  Part="4"
+AR Path="/57B6D511/57B6BA75/57B6437D" Ref="e59"  Part="4"
 F 0 "e59" H 2770 6000 60  0000 C CNN
 F 1 "MC10101" H 2790 5500 60  0000 C CNN
@@
 U 1 1 57B65227
 P 4500 2450
+AR Path="/57B68864/57B6BA75/57B65227" Ref="e57"  Part="1"
+AR Path="/57B6D511/57B6BA75/57B65227" Ref="e57"  Part="1"
 F 0 "e57" H 4520 3200 60  0000 C CNN
 F 1 "MC10164" H 4540 1700 60  0000 C CNN
@@
 U 1 1 57B66733
 P 6350 2450
+AR Path="/57B68864/57B6BA75/57B66733" Ref="e50"  Part="1"
+AR Path="/57B6D511/57B6BA75/57B66733" Ref="e50"  Part="1"
 F 0 "e50" H 6370 3200 60  0000 C CNN
 F 1 "MC10164" H 6390 1700 60  0000 C CNN
@@
 U 1 1 57B67599
 P 8200 2450
+AR Path="/57B68864/57B6BA75/57B67599" Ref="e43"  Part="1"
+AR Path="/57B6D511/57B6BA75/57B67599" Ref="e43"  Part="1"
 F 0 "e43" H 8220 3200 60  0000 C CNN
 F 1 "MC10164" H 8240 1700 60  0000 C CNN
@@
 U 1 1 57B687C3
 P 10050 2450
+AR Path="/57B68864/57B6BA75/57B687C3" Ref="e44"  Part="1"
+AR Path="/57B6D511/57B6BA75/57B687C3" Ref="e44"  Part="1"
 F 0 "e44" H 10070 3200 60  0000 C CNN
 F 1 "MC10164" H 10090 1700 60  0000 C CNN
@@
 U 1 1 57B68EF7
 P 11900 2450
+AR Path="/57B68864/57B6BA75/57B68EF7" Ref="e36"  Part="1"
+AR Path="/57B6D511/57B6BA75/57B68EF7" Ref="e36"  Part="1"
 F 0 "e36" H 11920 3200 60  0000 C CNN
 F 1 "MC10164" H 11940 1700 60  0000 C CNN
@@
 U 1 1 57B697CA
 P 13750 2450
+AR Path="/57B68864/57B6BA75/57B697CA" Ref="e37"  Part="1"
+AR Path="/57B6D511/57B6BA75/57B697CA" Ref="e37"  Part="1"
 F 0 "e37" H 13770 3200 60  0000 C CNN
 F 1 "MC10164" H 13790 1700 60  0000 C CNN
@@
 U 1 1 57B6B34B
 P 5550 4800
+AR Path="/57B68864/57B6BA75/57B6B34B" Ref="e69"  Part="1"
+AR Path="/57B6D511/57B6BA75/57B6B34B" Ref="e69"  Part="1"
 F 0 "e69" H 5570 5450 60  0000 C CNN
 F 1 "MC10147" H 5550 4600 60  0000 C CNN
@@
 U 1 1 57B6BFA9
 P 1900 6700
+AR Path="/57B68864/57B6BA75/57B6BFA9" Ref="U?"  Part="1"
+AR Path="/57B6D511/57B6BA75/57B6BFA9" Ref="U?"  Part="1"
 F 0 "U?" H 1920 6950 60  0000 C CNN
 F 1 "MC10105" H 1940 6450 60  0000 C CNN
@@
 U 2 1 57B6C012
 P 4250 6800
+AR Path="/57B68864/57B6BA75/57B6C012" Ref="U?"  Part="2"
+AR Path="/57B6D511/57B6BA75/57B6C012" Ref="U?"  Part="2"
 F 0 "U?" H 4270 7050 60  0000 C CNN
 F 1 "MC10105" H 4290 6550 60  0000 C CNN
@@
 NoConn ~ 1300 6800
 NoConn ~ 1300 6700
-Text Label 1300 6600 2    60   ~ 0
-dp04-clk
 NoConn ~ 4850 6700
 Wire Wire Line
@@
 U 1 1 57B6D95B
 P 3100 6500
+AR Path="/57B68864/57B6BA75/57B6D95B" Ref="DL1"  Part="1"
+AR Path="/57B6D511/57B6BA75/57B6D95B" Ref="DL1"  Part="1"
 F 0 "DL1" H 3100 6700 60  0000 C CNN
 F 1 "35ns" H 3100 6600 60  0000 C CNN
@@
 U 1 1 57B6DF9C
 P 7300 4800
+AR Path="/57B68864/57B6BA75/57B6DF9C" Ref="e70"  Part="1"
+AR Path="/57B6D511/57B6BA75/57B6DF9C" Ref="e70"  Part="1"
 F 0 "e70" H 7320 5450 60  0000 C CNN
 F 1 "MC10147" H 7300 4600 60  0000 C CNN
@@
 U 1 1 57B6E4E7
 P 9050 4800
+AR Path="/57B68864/57B6BA75/57B6E4E7" Ref="e71"  Part="1"
+AR Path="/57B6D511/57B6BA75/57B6E4E7" Ref="e71"  Part="1"
 F 0 "e71" H 9070 5450 60  0000 C CNN
 F 1 "MC10147" H 9050 4600 60  0000 C CNN
@@
 U 1 1 57B6EA16
 P 10800 4800
+AR Path="/57B68864/57B6BA75/57B6EA16" Ref="e72"  Part="1"
+AR Path="/57B6D511/57B6BA75/57B6EA16" Ref="e72"  Part="1"
 F 0 "e72" H 10820 5450 60  0000 C CNN
 F 1 "MC10147" H 10800 4600 60  0000 C CNN
@@
 U 1 1 57B6EE8E
 P 12550 4800
+AR Path="/57B68864/57B6BA75/57B6EE8E" Ref="e65"  Part="1"
+AR Path="/57B6D511/57B6BA75/57B6EE8E" Ref="e65"  Part="1"
 F 0 "e65" H 12570 5450 60  0000 C CNN
 F 1 "MC10147" H 12550 4600 60  0000 C CNN
@@
 U 1 1 57B6F292
 P 14300 4800
+AR Path="/57B68864/57B6BA75/57B6F292" Ref="e58"  Part="1"
+AR Path="/57B6D511/57B6BA75/57B6F292" Ref="e58"  Part="1"
 F 0 "e58" H 14320 5450 60  0000 C CNN
 F 1 "MC10147" H 14300 4600 60  0000 C CNN
@@
 U 1 1 57B6F81F
 P 12750 7300
+AR Path="/57B68864/57B6BA75/57B6F81F" Ref="e64"  Part="1"
+AR Path="/57B6D511/57B6BA75/57B6F81F" Ref="e64"  Part="1"
 F 0 "e64" H 12770 8000 60  0000 C CNN
 F 1 "MC10160" H 12790 6600 60  0000 C CNN
@@
 U 1 1 57B701A9
 P 2050 9250
+AR Path="/57B68864/57B6BA75/57B701A9" Ref="e38"  Part="1"
+AR Path="/57B6D511/57B6BA75/57B701A9" Ref="e38"  Part="1"
 F 0 "e38" H 2070 9500 60  0000 C CNN
 F 1 "MC10101" H 2090 9000 60  0000 C CNN
@@
 U 1 1 57B70692
 P 4150 8950
+AR Path="/57B68864/57B6BA75/57B70692" Ref="e61"  Part="1"
+AR Path="/57B6D511/57B6BA75/57B70692" Ref="e61"  Part="1"
 F 0 "e61" H 4170 9550 60  0000 C CNN
 F 1 "MC10141" H 4190 8350 60  0000 C CNN
@@
 U 1 1 57B71A9E
 P 5950 8950
+AR Path="/57B68864/57B6BA75/57B71A9E" Ref="e63"  Part="1"
+AR Path="/57B6D511/57B6BA75/57B71A9E" Ref="e63"  Part="1"
 F 0 "e63" H 5970 9550 60  0000 C CNN
 F 1 "MC10141" H 5990 8350 60  0000 C CNN
@@
 U 1 1 57B724AF
 P 7750 8950
+AR Path="/57B68864/57B6BA75/57B724AF" Ref="e8"  Part="1"
+AR Path="/57B6D511/57B6BA75/57B724AF" Ref="e8"  Part="1"
 F 0 "e8" H 7770 9550 60  0000 C CNN
 F 1 "MC10141" H 7790 8350 60  0000 C CNN
@@
 U 1 1 57B72C2C
 P 9650 8950
+AR Path="/57B68864/57B6BA75/57B72C2C" Ref="e10"  Part="1"
+AR Path="/57B6D511/57B6BA75/57B72C2C" Ref="e10"  Part="1"
 F 0 "e10" H 9670 9550 60  0000 C CNN
 F 1 "MC10141" H 9690 8350 60  0000 C CNN
@@
 Wire Bus Line
 	2500 1350 2400 1350
+Text HLabel 1300 6600 0    60   Input ~ 0
+dp04-clk
 $EndSCHEMATC

Commit message: DPA seems to be "done-ish"
Parts:
- gave numbers to parts that had none: 1
Connections:
- net ad.0 renamed ad.[n+0]
- net ad.1 renamed ad.[n+1]
- net ad.2 renamed ad.[n+2]
- net ad.3 renamed ad.[n+3]
- net ad.4 renamed ad.[n+4]
- net ad.5 renamed ad.[n+5]
- net adx.0 renamed adx.[n+0]
- net adx.1 renamed adx.[n+1]
- net adx.2 renamed adx.[n+2]
- net adx.3 renamed adx.[n+3]
- net adx.4 renamed adx.[n+4]
- net adx.5 renamed adx.[n+5]
- net apr-fm-adr.0 renamed apr-fm-adr.[n+0]
- net apr-fm-adr.1 renamed apr-fm-adr.[n+1]
- net apr-fm-adr.2 renamed apr-fm-adr.[n+2]
- net apr-fm-adr.3 renamed apr-fm-adr.[n+3]
- net apr-fm-block.0 renamed apr-fm-block.[n+0]
- net apr-fm-block.1 renamed apr-fm-block.[n+1]
- net apr-fm-block.2 renamed apr-fm-block.[n+2]
- net ar.0 renamed ar.[n+0]
- net ar.1 renamed ar.[n+1]
- net ar.2 renamed ar.[n+2]
- net ar.3 renamed ar.[n+3]
- net ar.4 renamed ar.[n+4]
- net ar.5 renamed ar.[n+5]
- net arx.0 renamed arx.[n+0]
- net arx.1 renamed arx.[n+1]
- net arx.2 renamed arx.[n+2]
- net arx.3 renamed arx.[n+3]
- net arx.4 renamed arx.[n+4]
- net arx.5 renamed arx.[n+5]
- net br.0 renamed br.[n+0]
- net br.1 renamed br.[n+1]
- net br.2 renamed br.[n+2]
- net br.3 renamed br.[n+3]
- net br.4 renamed br.[n+4]
- net br.5 renamed br.[n+5]
- net brx.0 renamed brx.[n+0]
- net brx.1 renamed brx.[n+1]
- net brx.2 renamed brx.[n+2]
- net brx.3 renamed brx.[n+3]
- net brx.4 renamed brx.[n+4]
- net brx.5 renamed brx.[n+5]
- net diag.4 renamed diag.[n+4]
- net diag.5 renamed diag.[n+5]
- net diag.6 renamed diag.[n+6]
- net ebus-d.0 renamed ebus-d.[n+0]
- net ebus-d.1 renamed ebus-d.[n+1]
- net ebus-d.2 renamed ebus-d.[n+2]
- net ebus-d.3 renamed ebus-d.[n+3]
- net ebus-d.4 renamed ebus-d.[n+4]
- net ebus-d.5 renamed ebus-d.[n+5]
- net ebus-driver-mask.0 renamed ebus-driver-mask.[n+0]
- net fm.0 renamed fm.[n+0]
- net fm.1 renamed fm.[n+1]
- net fm.2 renamed fm.[n+2]
- net fm.3 renamed fm.[n+3]
- net fm.4 renamed fm.[n+4]
- net fm.5 renamed fm.[n+5]
- net mq.0 renamed mq.[n+0]
- net mq.1 renamed mq.[n+1]
- net mq.2 renamed mq.[n+2]
- net mq.3 renamed mq.[n+3]
- net mq.4 renamed mq.[n+4]
- net mq.5 renamed mq.[n+5]

Commit message: Fix "last" [n...]
Connections:
- net ebus-driver-mask.[n+0] renamed [n/18+1,ctl-ad-to-ebus-l,ctl-ad-to-ebus-r]
Changed lines of the file:
@@
 NoConn ~ 3350 3550
 Text HLabel 1900 5850 0    60   Input ~ 0
-ebus-driver-mask.[n+0]
+[n/18+1,ctl-ad-to-ebus-l,ctl-ad-to-ebus-r]
 Text HLabel 1850 3550 0    60   Input ~ 0
 diag.[n+4]

Commit message: Update to kicad 5.1.2
Parts:
- DL1: symbol DELAYLINE -> o_ecl:DELAYLINE
- U1: symbol MC10105 -> o_ecl:MC10105
- e10, e61, e63, e8: symbol MC10141 -> o_ecl:MC10141
- e36, e37, e43, e44, e50, e57: symbol MC10164 -> o_ecl:MC10164
- e38, e59: symbol MC10101 -> o_ecl:MC10101
- e58, e65, e69, e70, e71, e72: symbol MC10147 -> o_ecl:MC10147
- e64: symbol MC10160 -> o_ecl:MC10160
Changed lines of the file:
@@
-EESchema Schematic File Version 2
-LIBS:o_ecl
-LIBS:ecl
-LIBS:power
-LIBS:device
-LIBS:transistors
-LIBS:conn
-LIBS:linear
-LIBS:regul
-LIBS:74xx
-LIBS:cmos4000
-LIBS:adc-dac
-LIBS:memory
-LIBS:xilinx
-LIBS:microcontrollers
-LIBS:dsp
-LIBS:microchip
-LIBS:analog_switches
-LIBS:motorola
-LIBS:texas
-LIBS:intel
-LIBS:audio
-LIBS:interface
-LIBS:digital-audio
-LIBS:philips
-LIBS:display
-LIBS:cypress
-LIBS:siliconi
-LIBS:opto
-LIBS:atmel
-LIBS:contrib
-LIBS:valves
+EESchema Schematic File Version 4
 LIBS:kl10-cache
-EELAYER 25 0
+EELAYER 30 0
 EELAYER END
 $Descr B 17000 11000
@@
 $EndDescr
 $Comp
-L MC10101 e59
+L o_ecl:MC10101 e59
 U 1 1 57B64287
 P 2750 3650
@@
 $EndComp
 $Comp
-L MC10101 e59
+L o_ecl:MC10101 e59
 U 2 1 57B6430A
 P 2750 4350
@@
 $EndComp
 $Comp
-L MC10101 e59
+L o_ecl:MC10101 e59
 U 3 1 57B64349
 P 2750 5050
@@
 $EndComp
 $Comp
-L MC10101 e59
+L o_ecl:MC10101 e59
 U 4 1 57B6437D
 P 2750 5750
@@
 diag-read-func-12x
 $Comp
-L MC10164 e57
+L o_ecl:MC10164 e57
 U 1 1 57B65227
 P 4500 2450
@@
 ebus-d.[n+0]
 $Comp
-L MC10164 e50
+L o_ecl:MC10164 e50
 U 1 1 57B66733
 P 6350 2450
@@
 ebus-d.[n+1]
 $Comp
-L MC10164 e43
+L o_ecl:MC10164 e43
 U 1 1 57B67599
 P 8200 2450
@@
 ebus-d.[n+2]
 $Comp
-L MC10164 e44
+L o_ecl:MC10164 e44
 U 1 1 57B687C3
 P 10050 2450
@@
 Connection ~ 7600 3050
 $Comp
-L MC10164 e36
+L o_ecl:MC10164 e36
 U 1 1 57B68EF7
 P 11900 2450
@@
 Connection ~ 9400 3050
 $Comp
-L MC10164 e37
+L o_ecl:MC10164 e37
 U 1 1 57B697CA
 P 13750 2450
@@
 Connection ~ 11300 3050
 $Comp
-L MC10147 e69
+L o_ecl:MC10147 e69
 U 1 1 57B6B34B
 P 5550 4800
@@
 apr-fm-adr.[n+0]
 $Comp
-L MC10105 U1
+L o_ecl:MC10105 U1
 U 1 1 57B6BFA9
 P 1900 6700
@@
 $EndComp
 $Comp
-L MC10105 U1
+L o_ecl:MC10105 U1
 U 2 1 57B6C012
 P 4250 6800
@@
 Connection ~ 4950 6200
 $Comp
-L DELAYLINE DL1
+L o_ecl:DELAYLINE DL1
 U 1 1 57B6D95B
 P 3100 6500
@@
 fm-write.0-35-l
 $Comp
-L MC10147 e70
+L o_ecl:MC10147 e70
 U 1 1 57B6DF9C
 P 7300 4800
@@
 	6700 6100 6700 5300
 $Comp
-L MC10147 e71
+L o_ecl:MC10147 e71
 U 1 1 57B6E4E7
 P 9050 4800
@@
 	6700 6100 13700 6100
 $Comp
-L MC10147 e72
+L o_ecl:MC10147 e72
 U 1 1 57B6EA16
 P 10800 4800
@@
 	10200 6100 10200 5300
 $Comp
-L MC10147 e65
+L o_ecl:MC10147 e65
 U 1 1 57B6EE8E
 P 12550 4800
@@
 Connection ~ 8450 6100
 $Comp
-L MC10147 e58
+L o_ecl:MC10147 e58
 U 1 1 57B6F292
 P 14300 4800
@@
 Connection ~ 11950 6100
 $Comp
-L MC10160 e64
+L o_ecl:MC10160 e64
 U 1 1 57B6F81F
 P 12750 7300
@@
 NoConn ~ 12150 7850
 $Comp
-L MC10101 e38
+L o_ecl:MC10101 e38
 U 1 1 57B701A9
 P 2050 9250
@@
 NoConn ~ 2650 9350
 $Comp
-L MC10141 e61
+L o_ecl:MC10141 e61
 U 1 1 57B70692
 P 4150 8950
@@
 br.[n+2]
 $Comp
-L MC10141 e63
+L o_ecl:MC10141 e63
 U 1 1 57B71A9E
 P 5950 8950
@@
 NoConn ~ 6550 8900
 $Comp
-L MC10141 e8
+L o_ecl:MC10141 e8
 U 1 1 57B724AF
 P 7750 8950
@@
 Connection ~ 5350 9300
 $Comp
-L MC10141 e10
+L o_ecl:MC10141 e10
 U 1 1 57B72C2C
 P 9650 8950
